File: Kicad_anool/speedo_odo_meter.kicad_pcb (KiCad board)
At the start: 2 copper layers, 12 parts, among them J1 Bat_3.0v, J2 AVR_SPI, J3 AudioJack4, SW1 SW_SPST, SW2 SW_SPST, U1 ATtiny85-20PU

Commit message: schematic and PCB layout complete
Parts:
- added C3: 100nf, speedo-odo-meter:C_Disc_D3.8mm_W2.6mm_P2.50mm, F.Cu at (111.2, 44.5)
- C1: footprint speedo-odo-meter:CP_Radial_D10.0mm_P2.50mm -> speedo-odo-meter:CP_Radial_D8.0mm_P2.50mm
- R1, R2, R3: footprint Resistor_THT:R_Axial_DIN0207_L6.3mm_D2.5mm_P7.62mm_Horizontal -> speedo-odo-meter:R_Axial_DIN0207_L6.3mm_D2.5mm_P7.62mm_Horizontal
- moved R1 47.9 mm to (108.5, 47.8)
- moved SW1 42.7 mm to (114.0, 68.0), turned to 180 degrees
- moved Brd1 36.7 mm to (120.0, 46.0)
- moved SW2 36.6 mm to (132.5, 68.0), turned to 180 degrees
- moved J3 32.1 mm to (131.5, 31.8), turned to 90 degrees
- moved U1 30.0 mm to (123.8, 50.8), turned to 270 degrees
- moved R3 19.2 mm to (128.0, 53.0), turned to 270 degrees
- moved J2 18.8 mm to (118.5, 62.5)
- moved C1 10.3 mm to (121.0, 41.5), turned to 270 degrees
- moved J1 9.93 mm to (127.2, 41.8), turned to 90 degrees
- moved R2 7.35 mm to (112.0, 53.0), turned to 270 degrees
- moved C2 6.76 mm to (127.2, 45.7), turned to 270 degrees
Routing:
- net +3V0: track 0.00 -> 100.2 mm
- net GND: track 0.00 -> 96.7 mm
- net SCK: track 0.00 -> 77.9 mm
- net MOSI: track 0.00 -> 53.4 mm
- net Reed_Output: track 0.00 -> 49.3 mm
- net RST: track 0.00 -> 41.6 mm
- net SW2: track 0.00 -> 33.4 mm
- net MISO: track 0.00 -> 27.4 mm
- added copper zone on B.Cu, net GND
Other:
- board outline added: 32 x 45 mm
- net class 0.40mm added: clearance 0.2, trace_width 0.4, via_dia 0.8, via_drill 0.4
- net class 1.00mm added: clearance 0.2, trace_width 1, via_dia 0.8, via_drill 0.4
- net class 2.00m added: clearance 0.2, trace_width 2, via_dia 0.8, via_drill 0.4
- board text added: "SPEEDO ODO METER"
