File: Kicad_anool/speedo_odo_meter.sch (KiCad schematic (older format))
At the start: 12 parts, among them J1 Bat_3.0v, J2 AVR_SPI, J3 AudioJack4, SW1 SW_SPST, SW2 SW_SPST, U1 ATtiny85-20PU

Commit message: schematic and PCB layout complete
Parts:
- added C3: 100nf, speedo-odo-meter:C_Disc_D3.8mm_W2.6mm_P2.50mm, symbol speedo_odo_meter:22PF-PTH-2.54MM-200V-5%-SparkFun-Capacitors
- C1: footprint speedo-odo-meter:CP_Radial_D10.0mm_P2.50mm -> speedo-odo-meter:CP_Radial_D8.0mm_P2.50mm
- R2: symbol Device:R -> speedo_odo_meter:R
Connections:
- net +3V0: now also J3.S; no longer J3.T
- net GND: now also C3.2
- net Reed_Output: now also J3.T, C3.1; no longer J3.S
Other:
- note added: "SERIAL PERIPHERAL INTERFACE (SPI)"
- note removed: "PROGRAMMING INTERFACE"
- moved on the sheet: Brd1, C1, C2, J1, J2, J3, R1, R3, SW1, SW2, U1
